Commit message: 20190722

File: ros_package/cheetah_description/urdf/cheetah_old.urdf (robot description, URDF)
Before this commit: robot cheetah, 13 links, 12 joints
Links:
- link LB2: mass 0.323696605188412 -> 0.323696605007919
- link LB3: mass 0.13341 -> 0.114240539936642
- link LF1: mass 0.128744524052319 -> 0.12874452405232
- link LF2: mass 0.323696829552903 -> 0.323696832719431
- link LF3: mass 0.13341 -> 0.114240540212022
- link RB1: mass 0.128744524870708 -> 0.128744524870709
- link RB2: mass 0.323696977049233 -> 0.323696976849496
- link RB3: mass 0.13341 -> 0.114240538818722
- link RF1: mass 0.128744523661008 -> 0.128744523661006
- link RF2: mass 0.293729852554546 -> 0.293729852808938
- link RF3: mass 0.13341 -> 0.114240539524017
Joints:
- joint LB_JOINT1: axis 0 1 0 -> 0 0 -1; origin xyz=-0.173599224631526 0 0.0725529089199335 rpy=-1.88165997540291E-15 -8.49741356322415E-31 1.38777878078145E-14 -> xyz=0.173599224631526 0 0.0725529089199335 rpy=-1.57079632679489 -0.550782542641248 3.7606585259785E-17
- joint LB_JOINT2: axis 0.999630540713182 0 0.0271805458641196 -> 0.999999999999992 0 0; origin xyz=-0.0276897658681326 -0.0359335135474832 0.000752902296081187 rpy=0 0 0 -> xyz=0.0239889055485236 0.0138499967714876 0.0359335135116864 rpy=-2.80449724784631 6.30450004185909E-15 0.523598766712586
- joint LB_JOINT3: axis 0.999630540713182 0 0.0271805458641197 -> 0 0 1; origin xyz=-0.0493319949518443 -0.0969348369953719 -0.218293046902893 rpy=0 0 0 -> xyz=0.0433804661279571 -0.239257600341479 -0.0188626161448396 rpy=-1.57079645284584 1.2337009210514 -1.57079632679494
- joint LF_JOINT1: axis 0 1 0 -> 0 0 1; origin xyz=-0.173599224631532 0.399354557389219 0.0725529089199334 rpy=-1.60410421924662E-15 -9.17720664828209E-31 1.49880108324396E-14 -> xyz=0.173599224631532 -0.399354557389219 0.0725529089199334 rpy=1.5707963267949 0.511092050822873 -3.43375535468868E-17
- joint LF_JOINT2: axis 1 0 0 -> 0 0 0.99999999999998; origin xyz=-0.0276978335511204 0.0707119289660939 0.000346434087151945 rpy=0 0.0125069428080353 0 -> xyz=0.0239889006854609 0.0138500051937306 0.0707119290859076 rpy=1.5707963267949 -0.368671500214442 2.09439511787625
- joint LF_JOINT3: axis 0.999921789331814 0 0.0125066070324357 -> 0 0 1; origin xyz=-0.0433804402006036 -0.141483529247529 -0.193861834684897 rpy=0 -0.0125069428080353 0 -> xyz=-0.231822995878655 -0.0621135670258962 0.0433804774370614 rpy=-2.01086507658697E-07 5.47983968079473E-15 -1.93946782700934
- joint RB_JOINT1: axis 0 1 0 -> 0 0 -1; origin xyz=-0.0535992246315264 0 0.0725529089199335 rpy=-1.60538682552622E-15 -0.0399761301393608 1.40807257464315E-14 -> xyz=0.0535992246315264 0 0.0725529089199335 rpy=1.57079632679489 0.483622535977452 -3.14159265358979
- joint RB_JOINT2: axis 1 0 0 -> 0 0 0.999999999999996; origin xyz=0.0277000009004106 -0.0359335144587992 0 rpy=0 -9.71536796845474E-09 0 -> xyz=0.0239889051808841 0.0138499974087561 0.0359335135244585 rpy=1.57079632679491 0.692488919582274 2.09439507785289
- joint RB_JOINT3: axis 0.999201060527875 0 0.0399654931155527 -> 0 0 1; origin xyz=0.0433804375529314 -0.100202218464516 -0.218081441703766 rpy=0 0.0399761398547287 0 -> xyz=-0.231823006662634 -0.0621135667231729 0.0433804202483734 rpy=-2.18941904487291E-15 -8.34781210545811E-08 0.692488919581947
- joint RF_JOINT1: axis 0 1 0 -> 0 0 1; origin xyz=-0.053599224631532 0.399354557389219 0.0725529089199333 rpy=-1.0489927069341E-15 3.53125934784206E-07 1.41553431935442E-14 -> xyz=0.053599224631532 -0.399354557389219 0.0725529089199333 rpy=-1.5707963267949 -0.523598601027881 3.14159265358979
- joint RF_JOINT2: axis 0.999999999999882 0 0 -> 0 0 0.99999999999992; origin xyz=0.0277000007048783 0.0707119290863223 0 rpy=0 -9.71536797770656E-09 0 -> xyz=0.0239889012320922 0.0138500042482511 0.070711929086322 rpy=-1.57079632679487 -0.863675085440379 -1.04719753259462
- joint RF_JOINT3: axis 0.999999999999882 0 0 -> 0 0 0.999999999999876; origin xyz=0.0433804384533972 -0.135888064174125 -0.197824250345348 rpy=0 -2.79819504647401E-16 0 -> xyz=-0.231823008442479 -0.0621135692653797 0.0433804071002776 rpy=1.58490470087489E-07 -4.8795080220757E-16 -0.707121241354518
